File: Hardware/PCB/Elo_112.kicad_pcb (KiCad board)
At the start: 2 copper layers, 0 parts

Commit message: Add files via upload
Parts:
- added C1: 100nF, Capacitor_SMD:C_0402_1005Metric, B.Cu at (78.4, 97.1)
- added C10: 4.7nF, Capacitor_SMD:C_0402_1005Metric, F.Cu at (73.8, 98.0)
- added C11: 100nF, Capacitor_SMD:C_0402_1005Metric, F.Cu at (91.5, 98.7)
- added C12: 4.7uF, Capacitor_SMD:C_0402_1005Metric, B.Cu at (67.5, 101.6)
- added C13: 4.7uF, Capacitor_SMD:C_0402_1005Metric, B.Cu at (91.9, 94.9)
- added C18: 100nF, Capacitor_SMD:C_0402_1005Metric, F.Cu at (87.5, 97.7)
- added C2: 100nF, Capacitor_SMD:C_0402_1005Metric, F.Cu at (77.4, 97.1)
- added C22: 22u, Capacitor_SMD:C_0402_1005Metric, F.Cu at (78.8, 106.5)
- added C23: 22u, Capacitor_SMD:C_0402_1005Metric, F.Cu at (78.8, 108.9)
- added C3: 100nF, Capacitor_SMD:C_0402_1005Metric, F.Cu at (76.4, 97.1)
- added C4: 100nF, Capacitor_SMD:C_0402_1005Metric, F.Cu at (75.4, 97.1)
- added C41: 100n, Capacitor_SMD:C_0402_1005Metric, F.Cu at (68.3, 97.8)
- added C5: 4.7uF, Capacitor_SMD:C_0402_1005Metric, B.Cu at (79.5, 97.1)
- added C6: 1 uF, Capacitor_SMD:C_0402_1005Metric, F.Cu at (87.5, 99.7)
- added C7: 10nF, Capacitor_SMD:C_0402_1005Metric, F.Cu at (87.5, 101.6)
- added C8: 4.7uF, Capacitor_SMD:C_0402_1005Metric, B.Cu at (80.9, 103.8)
- added C9: 4.7uF, Capacitor_SMD:C_0402_1005Metric, F.Cu at (89.1, 95.2)
- added D1: LED, LED_SMD:LED_0402_1005Metric, F.Cu at (98.9, 88.2)
- added D10: LED, LED_SMD:LED_0402_1005Metric, F.Cu at (96.8, 86.9)
- added D11: LED, LED_SMD:LED_0402_1005Metric, F.Cu at (96.8, 85.7)
- added D12: LED, LED_SMD:LED_0402_1005Metric, F.Cu at (96.8, 84.4)
- added D13: LED, LED_SMD:LED_0402_1005Metric, F.Cu at (96.8, 83.2)
- added D14: LED, LED_SMD:LED_0402_1005Metric, F.Cu at (96.8, 81.9)
- added D15: LED, LED_SMD:LED_0402_1005Metric, F.Cu at (96.8, 80.7)
- added D16: LED, LED_SMD:LED_0402_1005Metric, F.Cu at (96.8, 79.4)
- added D17: LED, LED_SMD:LED_0402_1005Metric, F.Cu at (94.7, 88.2)
- added D18: LED, LED_SMD:LED_0402_1005Metric, F.Cu at (94.7, 86.9)
- added D19: LED, LED_SMD:LED_0402_1005Metric, F.Cu at (94.7, 85.7)
- added D2: LED, LED_SMD:LED_0402_1005Metric, F.Cu at (98.9, 86.9)
- added D20: LED, LED_SMD:LED_0402_1005Metric, F.Cu at (94.7, 84.4)
- added D21: LED, LED_SMD:LED_0402_1005Metric, F.Cu at (94.7, 83.2)
- added D22: LED, LED_SMD:LED_0402_1005Metric, F.Cu at (94.7, 81.9)
- added D23: LED, LED_SMD:LED_0402_1005Metric, F.Cu at (94.7, 80.7)
- added D24: LED, LED_SMD:LED_0402_1005Metric, F.Cu at (94.7, 79.4)
- added D25: LED, LED_SMD:LED_0402_1005Metric, F.Cu at (92.6, 88.2)
- added D26: LED, LED_SMD:LED_0402_1005Metric, F.Cu at (92.6, 86.9)
- added D27: LED, LED_SMD:LED_0402_1005Metric, F.Cu at (92.6, 85.7)
- added D28: LED, LED_SMD:LED_0402_1005Metric, F.Cu at (92.6, 84.4)
- added D29: LED, LED_SMD:LED_0402_1005Metric, F.Cu at (92.6, 83.2)
- added D3: LED, LED_SMD:LED_0402_1005Metric, F.Cu at (98.9, 85.7)
- added D30: LED, LED_SMD:LED_0402_1005Metric, F.Cu at (92.6, 81.9)
- added D31: LED, LED_SMD:LED_0402_1005Metric, F.Cu at (92.6, 80.7)
- added D32: LED, LED_SMD:LED_0402_1005Metric, F.Cu at (92.6, 79.4)
- added D33: LED, LED_SMD:LED_0402_1005Metric, F.Cu at (90.5, 88.2)
- added D34: LED, LED_SMD:LED_0402_1005Metric, F.Cu at (90.5, 86.9)
- added D35: LED, LED_SMD:LED_0402_1005Metric, F.Cu at (90.5, 85.7)
- added D36: LED, LED_SMD:LED_0402_1005Metric, F.Cu at (90.5, 84.4)
- added D37: LED, LED_SMD:LED_0402_1005Metric, F.Cu at (90.5, 83.2)
- added D38: LED, LED_SMD:LED_0402_1005Metric, F.Cu at (90.5, 81.9)
- added D39: LED, LED_SMD:LED_0402_1005Metric, F.Cu at (90.5, 80.7)
- added D4: LED, LED_SMD:LED_0402_1005Metric, F.Cu at (98.9, 84.4)
- added D40: LED, LED_SMD:LED_0402_1005Metric, F.Cu at (90.5, 79.4)
- added D41: LED, LED_SMD:LED_0402_1005Metric, F.Cu at (88.4, 88.2)
- added D42: LED, LED_SMD:LED_0402_1005Metric, F.Cu at (88.4, 86.9)
- added D43: LED, LED_SMD:LED_0402_1005Metric, F.Cu at (88.4, 85.7)
- added D44: LED, LED_SMD:LED_0402_1005Metric, F.Cu at (88.4, 84.4)
- added D45: LED, LED_SMD:LED_0402_1005Metric, F.Cu at (88.4, 83.2)
- added D46: LED, LED_SMD:LED_0402_1005Metric, F.Cu at (88.4, 81.9)
- added D47: LED, LED_SMD:LED_0402_1005Metric, F.Cu at (88.4, 80.7)
- added D48: LED, LED_SMD:LED_0402_1005Metric, F.Cu at (88.4, 79.4)
- added D49: LED, LED_SMD:LED_0402_1005Metric, F.Cu at (86.3, 88.2)
- added D5: LED, LED_SMD:LED_0402_1005Metric, F.Cu at (98.9, 83.2)
- added D50: LED, LED_SMD:LED_0402_1005Metric, F.Cu at (86.3, 86.9)
- added D51: LED, LED_SMD:LED_0402_1005Metric, F.Cu at (86.3, 85.7)
- added D52: LED, LED_SMD:LED_0402_1005Metric, F.Cu at (86.3, 84.4)
- added D53: LED, LED_SMD:LED_0402_1005Metric, F.Cu at (86.3, 83.2)
- added D54: LED, LED_SMD:LED_0402_1005Metric, F.Cu at (86.3, 81.9)
- added D55: LED, LED_SMD:LED_0402_1005Metric, F.Cu at (86.3, 80.7)
- added D56: LED, LED_SMD:LED_0402_1005Metric, F.Cu at (86.3, 79.4)
- added D57: LED, LED_SMD:LED_0402_1005Metric, F.Cu at (84.2, 88.2)
- added D58: LED, LED_SMD:LED_0402_1005Metric, F.Cu at (84.2, 86.9)
- added D59: LED, LED_SMD:LED_0402_1005Metric, F.Cu at (84.2, 85.7)
- added D6: LED, LED_SMD:LED_0402_1005Metric, F.Cu at (98.9, 81.9)
- added D60: LED, LED_SMD:LED_0402_1005Metric, F.Cu at (84.2, 84.4)
- added D61: LED, LED_SMD:LED_0402_1005Metric, F.Cu at (84.2, 83.2)
- added D62: LED, LED_SMD:LED_0402_1005Metric, F.Cu at (84.2, 81.9)
- added D63: LED, LED_SMD:LED_0402_1005Metric, F.Cu at (84.2, 80.7)
- added D64: LED, LED_SMD:LED_0402_1005Metric, F.Cu at (84.2, 79.4)
- added D65: 1N5817, Diode_SMD:D_SOD-123, F.Cu at (75.4, 103.1)
- added D66: ESD3.3, Diode_SMD:SODFL1006X40N, F.Cu at (87.4, 96.6)
- added D67: Green, LED_SMD:LED_0805_2012Metric, B.Cu at (92.6, 112.0)
- added D68: ESD3.3, Diode_SMD:SODFL1006X40N, F.Cu at (91.5, 100.4)
- added D7: LED, LED_SMD:LED_0402_1005Metric, F.Cu at (98.9, 80.7)
- added D8: LED, LED_SMD:LED_0402_1005Metric, F.Cu at (98.9, 79.4)
- added D9: LED, LED_SMD:LED_0402_1005Metric, F.Cu at (96.8, 88.2)
- added F1: Polyfuse 1A, Fuse:FUSC1608X100N, F.Cu at (70.0, 103.0)
- added FB1: BLM21PG220, Diode_SMD:IND_BLM21_MUR-L, F.Cu at (72.0, 103.1)
- added J1: USB_C_Receptacle_USB2.0_16P, Connector_USB:USB_C_Receptacle_HCTL_HC-TYPE-C-16P-01A, B.Cu at (71.1, 110.7)
- added Q1: PNP, Package_TO_SOT_SMD:SOT-23, F.Cu at (98.4, 94.6)
- added Q10: MMBT2222A, Package_TO_SOT_SMD:SOT-23, F.Cu at (78.5, 82.2)
- added Q11: MMBT2222A, Package_TO_SOT_SMD:SOT-23, B.Cu at (75.0, 82.2)
- added Q12: MMBT2222A, Package_TO_SOT_SMD:SOT-23, F.Cu at (75.0, 82.2)
- added Q13: MMBT2222A, Package_TO_SOT_SMD:SOT-23, B.Cu at (71.4, 82.2)
- added Q14: MMBT2222A, Package_TO_SOT_SMD:SOT-23, F.Cu at (71.4, 82.2)
- added Q15: MMBT2222A, Package_TO_SOT_SMD:SOT-23, B.Cu at (67.9, 82.2)
- added Q16: MMBT2222A, Package_TO_SOT_SMD:SOT-23, F.Cu at (67.9, 82.2)
- added Q2: PNP, Package_TO_SOT_SMD:SOT-23, B.Cu at (98.4, 94.6)
- added Q3: PNP, Package_TO_SOT_SMD:SOT-23, F.Cu at (98.4, 98.0)
- added Q4: PNP, Package_TO_SOT_SMD:SOT-23, B.Cu at (98.4, 98.0)
- added Q5: PNP, Package_TO_SOT_SMD:SOT-23, F.Cu at (98.4, 101.5)
- added Q6: PNP, Package_TO_SOT_SMD:SOT-23, B.Cu at (98.4, 101.5)
- added Q7: PNP, Package_TO_SOT_SMD:SOT-23, F.Cu at (98.4, 104.9)
- added Q8: PNP, Package_TO_SOT_SMD:SOT-23, B.Cu at (98.4, 104.9)
- added Q9: MMBT2222A, Package_TO_SOT_SMD:SOT-23, B.Cu at (78.5, 82.2)
- added R1: 5.1k, Resistor_SMD:R_0402_1005Metric, B.Cu at (72.4, 102.5)
- added R10: R_Small, Resistor_SMD:R_0402_1005Metric, F.Cu at (80.7, 96.2)
- added R11: R_Small, Resistor_SMD:R_0402_1005Metric, F.Cu at (80.9, 89.0)
- added R12: R_Small, Resistor_SMD:R_0402_1005Metric, F.Cu at (81.5, 91.4)
- added R13: R_Small, Resistor_SMD:R_0402_1005Metric, B.Cu at (83.8, 88.8)
- added R14: R_Small, Resistor_SMD:R_0402_1005Metric, B.Cu at (85.8, 88.8)
- added R15: R_Small, Resistor_SMD:R_0402_1005Metric, B.Cu at (87.9, 88.7)
- added R16: R_Small, Resistor_SMD:R_0402_1005Metric, B.Cu at (90.0, 88.7)
- added R17: R_Small, Resistor_SMD:R_0402_1005Metric, B.Cu at (92.1, 88.7)
- added R18: R_Small, Resistor_SMD:R_0402_1005Metric, B.Cu at (94.2, 88.7)
- added R19: R_Small, Resistor_SMD:R_0402_1005Metric, B.Cu at (96.3, 88.7)
- added R2: 5.1k, Resistor_SMD:R_0402_1005Metric, B.Cu at (69.4, 102.5)
- added R20: R_Small, Resistor_SMD:R_0402_1005Metric, B.Cu at (98.4, 88.7)
- added R23: 1k, Resistor_SMD:R_0402_1005Metric, B.Cu at (89.8, 112.0)
- added R3: 100Ohm, Resistor_SMD:R_0402_1005Metric, F.Cu at (86.0, 99.6)
- added R4: 5.1KOhm, Resistor_SMD:R_0402_1005Metric, F.Cu at (84.9, 99.5)
- added R5: R_Small, Resistor_SMD:R_0402_1005Metric, F.Cu at (78.2, 91.5)
- added R6: R_Small, Resistor_SMD:R_0402_1005Metric, F.Cu at (78.7, 88.9)
- added R7: R_Small, Resistor_SMD:R_0402_1005Metric, F.Cu at (76.7, 86.4)
- added R8: R_Small, Resistor_SMD:R_0402_1005Metric, F.Cu at (74.3, 85.9)
- added R9: R_Small, Resistor_SMD:R_0402_1005Metric, F.Cu at (74.6, 84.9)
- added SW1: RESET, Button_Switch_SMD:SW_CS1213AGF260_CRS, B.Cu at (89.3, 107.5)
- added SW2: RESET, Button_Switch_SMD:SW_CS1213AGF260_CRS, B.Cu at (93.0, 107.5)
- added U1: STM32F103C8Tx, Package_QFP:LQFP-48_7x7mm_P0.5mm, B.Cu at (85.2, 99.4)
- added U2: CH340G, Package_SO:SOIC-16_3.9x9.9mm_P1.27mm, B.Cu at (72.4, 93.0)
- added U4: LM1117MP-ADJ, Regulator:DCY0004A_L, B.Cu at (83.3, 109.3)
- added U6: USBLC6-4SC6, Package_TO_SOT_SMD:SOT-23-6, F.Cu at (71.1, 98.2)
- added Y1: ASE-8MHz, Oscillator:Oscillator_SMD_Abracon_ASE-4Pin_3.2x2.5mm, B.Cu at (92.2, 97.5)
- added Y3: ASE-12MHz, Oscillator:Oscillator_SMD_Abracon_ASE-4Pin_3.2x2.5mm, B.Cu at (67.2, 99.1)
Routing:
- net GND: track 0.00 -> 79.4 mm, vias 0 -> 36
- net Net-(D1-K): track 0.00 -> 44.1 mm, vias 0 -> 2
- net Net-(D10-K): track 0.00 -> 43.8 mm, vias 0 -> 2
- net +3V3: track 0.00 -> 43.8 mm, vias 0 -> 16
- net Net-(D12-K): track 0.00 -> 41.7 mm, vias 0 -> 1
- net Net-(D11-K): track 0.00 -> 41.6 mm, vias 0 -> 2
- net Net-(D14-K): track 0.00 -> 41.2 mm, vias 0 -> 2
- net Net-(D13-K): track 0.00 -> 39.5 mm, vias 0 -> 2
- net Net-(D15-K): track 0.00 -> 37.1 mm, vias 0 -> 2
- net Net-(D16-K): track 0.00 -> 37.1 mm, vias 0 -> 1
- net /P_5: track 0.00 -> 35.6 mm, vias 0 -> 1
- net /P_4: track 0.00 -> 35.2 mm, vias 0 -> 2
- net /P_7: track 0.00 -> 34.9 mm, vias 0 -> 1
- net /P_6: track 0.00 -> 34.9 mm, vias 0 -> 2
- net /P_8: track 0.00 -> 34.6 mm, vias 0 -> 3
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- added copper zone on In2.Cu, net +3V3
- added copper zone on In1.Cu, net GND
Other:
- board outline added: 35 x 35 mm
- copper layers 2 -> 4
