File: Hardware/PCB/Elo_112.kicad_pcb (KiCad board)
At the start: 4 copper layers, 35 x 35 mm, 133 parts, among them J1 USB_C_Receptacle_USB2.0_16P, Q1 PNP, Q10 MMBT2222A, Q11 MMBT2222A, Q12 MMBT2222A, Q13 MMBT2222A, Q14 MMBT2222A, Q15 MMBT2222A, Q16 MMBT2222A, Q2 PNP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

Commit message: Add files via upload
Parts:
- removed C13: 4.7uF, Capacitor_SMD:C_0402_1005Metric
- removed Y3: ASE-12MHz, Oscillator:Oscillator_SMD_Abracon_ASE-4Pin_3.2x2.5mm
- added C14: 33pF, Capacitor_SMD:C_0402_1005Metric, B.Cu at (91.3, 97.9)
- added C15: 33pF, Capacitor_SMD:C_0402_1005Metric, B.Cu at (93.2, 98.5)
- added C16: 15pF, Capacitor_SMD:C_0402_1005Metric, B.Cu at (66.5, 98.2)
- added R21: 100 Ohm, Resistor_SMD:R_0402_1005Metric, B.Cu at (91.3, 98.9)
- added R22: 100 Ohm, Resistor_SMD:R_0402_1005Metric, B.Cu at (67.9, 97.6)
- added Y2: 8MHz, Crystal:Crystal_SMD_3225-4Pin_3.2x2.5mm, B.Cu at (92.2, 95.2)
- C12: value 4.7uF -> 15pF
- Y1: value ASE-8MHz -> 12MHz; footprint Oscillator:Oscillator_SMD_Abracon_ASE-4Pin_3.2x2.5mm -> Crystal:Crystal_SMD_3225-4Pin_3.2x2.5mm
- moved Y1 24.8 mm to (67.7, 101.3), turned to 180 degrees
- moved C12 4.50 mm to (69.7, 97.7), turned to 0 degrees
- moved R2 1.91 mm to (70.1, 104.3)
Connections:
- C12 pad 1: +3V3 -> /Xtal_in_1
- U1 pad 5: Net-(U1-PD0) -> /Xtal_in_2
- U1 pad 6: unconnected-(U1-PD1-Pad6) -> /Xtal_out_2
- U2 pad 7: Net-(U2-XI) -> /Xtal_in_1
- U2 pad 8: unconnected-(U2-XO-Pad8) -> /Xtal_out_1
- Y1 pad 1: +3V3 -> /Xtal_in_1
- Y1 pad 3: Net-(U1-PD0) -> Net-(C16-Pad1)
- Y1 pad 4: +3V3 -> GND
Routing:
- net GND: track 79.4 -> 90.2 mm, vias 36 -> 37
- net +3V3: track 43.8 -> 34.7 mm, vias 16 -> 14
- net /Xtal_in_1: track 0.00 -> 7.55 mm
- net Net-(C15-Pad1): track 0.00 -> 7.16 mm
- net /Xtal_in_2: track 0.00 -> 7.12 mm
- net Net-(C16-Pad1): track 0.00 -> 6.33 mm
- net Net-(U2-XI): track 3.05 -> 0.00 mm
- net Net-(U1-PD0): track 2.05 -> 0.00 mm
- net /Xtal_out_1: track 0.00 -> 1.65 mm
- net /Xtal_out_2: track 0.00 -> 1.50 mm
- net /CC2_2: track 3.98 -> 2.52 mm
- net Net-(Q8-E): track 29.2 -> 29.7 mm
- net Net-(Q7-E): track 26.6 -> 27.1 mm
