File: Hardware/PCB/Elo_112.kicad_sch (KiCad schematic)
At the start: 117 parts, among them J1 USB_C_Receptacle_USB2.0_16P, Q1 MMBT2222A, Q10 MMBT2222A, Q11 MMBT2222A, Q12 MMBT2222A, Q13 MMBT2222A, Q14 MMBT2222A, Q15 MMBT2222A, Q16 MMBT2222A, Q2 MMBT2222A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

Commit message: Add files via upload
Parts:
- removed Q1, Q2, Q3, Q4, Q5, Q6, Q7, Q8: MMBT2222A, Package_TO_SOT_SMD:SOT-23, symbol Transistor_BJT:MMBT2222A
- added Q1, Q2, Q3, Q4, Q5, Q6, Q7, Q8: PNP, Package_TO_SOT_SMD:SOT-23, symbol Simulation_SPICE:PNP
- added R10, R11, R12, R13, R14, R15, R16, R17, R18, R19, R20, R5, R6, R7, R8, R9: R_Small, Resistor_SMD:R_0402_1005Metric, symbol Device:R_Small
Connections:
- net +3V3: now also Q1.2 (B), Q2.2 (B), Q3.2 (B), Q4.2 (B), Q5.2 (B), Q6.2 (B), Q7.2 (B), Q8.2 (B)
- net G_1: now also R5.2; no longer Q16.1 (B)
- net G_2: now also R6.2; no longer Q15.1 (B)
- net G_3: now also R7.2; no longer Q14.1 (B)
- net G_4: now also R8.2; no longer Q13.1 (B)
- net G_5: now also R9.2; no longer Q12.1 (B)
- net G_6: now also R10.2; no longer Q11.1 (B)
- net G_7: now also R11.2; no longer Q10.1 (B)
- net G_8: now also R12.2; no longer Q9.1 (B)
- net P_1: now also Q1.1 (C)
- net P_2: now also Q2.1 (C)
- net P_3: now also Q3.1 (C)
- net P_4: now also Q4.1 (C)
- net P_5: now also Q5.1 (C)
- net P_6: now also Q6.1 (C)
- net P_7: now also Q7.1 (C)
- net P_8: now also Q8.1 (C)
- net at D33.2 (A), D34.2 (A), D35.2 (A)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: now also R16.2
- net at D1.2 (A), D2.2 (A), D3.2 (A)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: now also R20.2
- net at D57.2 (A), D58.2 (A), D59.2 (A)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: now also R13.2
- net at D17.2 (A), D18.2 (A), D19.2 (A)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: now also R18.2
- net at D41.2 (A), D42.2 (A), D43.2 (A)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: now also R15.2
- net at D25.2 (A), D26.2 (A), D27.2 (A)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: now also R17.2
- net at D10.2 (A), D11.2 (A), D12.2 (A)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: now also R19.2
- net at D49.2 (A), D50.2 (A), D51.2 (A)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: now also R14.2
- new net: Q12.1 (B), R9.1
- new net: Q9.1 (B), R12.1
- new net: Q15.1 (B), R6.1
- new net: Q5.3 (E), R16.1
- new net: Q7.3 (E), R14.1
- new net: Q13.1 (B), R8.1
- new net: Q16.1 (B), R5.1
- new net: Q11.1 (B), R10.1
- new net: Q14.1 (B), R7.1
- new net: Q4.3 (E), R17.1
- new net: Q3.3 (E), R18.1
- new net: Q2.3 (E), R19.1
- new net: Q10.1 (B), R11.1
- new net: Q8.3 (E), R13.1
- new net: Q1.3 (E), R20.1
- new net: Q6.3 (E), R15.1

Commit message: Add files via upload
Parts:
- removed C13: 4.7uF, Capacitor_SMD:C_0402_1005Metric, symbol Device:C_Small
- removed Y1: ASE-8MHz, Oscillator:Oscillator_SMD_Abracon_ASE-4Pin_3.2x2.5mm, symbol Oscillator:ASE-xxxMHz
- removed Y3: ASE-12MHz, Oscillator:Oscillator_SMD_Abracon_ASE-4Pin_3.2x2.5mm, symbol Oscillator:ASE-xxxMHz
- added C14, C15, C16: 33pF, symbol Device:C_Small
- added R21, R22: 100 Ohm, symbol Device:R_Small
- added Y1: 12MHz, symbol Device:Crystal_GND24_Small
- added Y2: 8MHz, symbol Device:Crystal_GND24_Small
- C12: value 4.7uF -> 33pF; footprint Capacitor_SMD:C_0402_1005Metric -> (none)
Connections:
- net +3V3: no longer C12.1
- net GND: now also C14.2, C15.2, C16.2, Y1.2, Y1.4, Y2.2, Y2.4
- net Xtal_in: now reaches U2.7 (XI)
- net Xtal_in: now also C12.1, U1.5 (PD0), C14.1, Y1.1, Y2.1
- net Xtal_out: now reaches U2.8 (XO)
- net Xtal_out: now also U1.6 (PD1), R21.2, R22.2
- new net: C15.1, R21.1, Y2.3
- new net: C16.1, R22.1, Y1.3
Other:
- note added: "1]The PNP BJT symbol is intentionally different. I did not want to create a custom schematic symbol, so I used the standard symbol that strictly follows the datasheet. Therefore, this should not be treated as a fault. It directly corresponds to the "MMBT2907A" transistor."
- note added: "2]The Capacitor values for the Crystals are yet to be calculated they will be updated in the datasheet"
- note added: "Buttons_STM32"
- note added: "CH350G"
- note added: "Crystal_CH350G"
- note added: "Crystal_STM32"
- note added: "Important Note"
- note added: "LED_Matrix"
- note added: "STM_32"
- note added: "USB_C + ESD_P"
- moved on the sheet: C1, C10, C11, C18, C2, C22, C23, C3, C4, C41, C5, C6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

Commit message: Add files via upload
Parts:
- C12, C16: value 33pF -> 15pF; footprint (none) -> Capacitor_SMD:C_0402_1005Metric
- C14, C15: footprint (none) -> Capacitor_SMD:C_0402_1005Metric
- R21, R22: footprint (none) -> Resistor_SMD:R_0402_1005Metric
- Y1, Y2: footprint (none) -> Crystal:Crystal_SMD_3225-4Pin_3.2x2.5mm
Connections:
- net Xtal_in renamed Xtal_in_1
- net Xtal_in_1: no longer C14.1, U1.5 (PD0), Y2.1
- net Xtal_out renamed Xtal_out_1
- net Xtal_out_1: no longer R21.2, U1.6 (PD1)
- new net Xtal_in_2: C14.1, U1.5 (PD0), Y2.1
- new net Xtal_out_2: R21.2, U1.6 (PD1)
Other:
- note added: "3] The LM1117-ADJ is used but is LM1117 3.3 with the correct schematic it will be updated in the datasheet for further use"
Changed lines of the file:
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@@
 		)
 	)
+	(text "3] The LM1117-ADJ is used but is LM1117 3.3 with the correct \nschematic it will be updated in the datasheet for further use"
+		(exclude_from_sim no)
+		(at 296.926 198.12 0)
+		(effects
+			(font
+				(size 1.778 1.778)
+			)
+			(justify left)
+		)
+	)
 	(text "Buttons_STM32"
 		(exclude_from_sim no)
@@
 	(wire
 		(pts
-			(xy 316.23 81.28) (xy 325.12 81.28)
+			(xy 313.69 81.28) (xy 325.12 81.28)
 		)
 		(stroke
@@
 	(wire
 		(pts
-			(xy 316.23 83.82) (xy 325.12 83.82)
+			(xy 313.69 83.82) (xy 325.12 83.82)
 		)
 		(stroke
@@
 		)
 	)
-	(label "Xtal_in"
+	(label "Xtal_in_2"
 		(at 125.73 247.65 0)
 		(effects
@@
 		)
 	)
-	(label "Xtal_in"
+	(label "Xtal_in_1"
 		(at 194.31 173.99 0)
 		(effects
@@
 		)
 	)
-	(label "Xtal_out"
-		(at 316.23 83.82 0)
+	(label "Xtal_out_2"
+		(at 313.69 83.82 0)
 		(effects
 			(font
@@
 		)
 	)
-	(label "Xtal_out"
+	(label "Xtal_out_1"
 		(at 194.31 185.42 0)
 		(effects
@@
 		)
 	)
-	(label "Xtal_in"
-		(at 316.23 81.28 0)
+	(label "Xtal_in_2"
+		(at 313.69 81.28 0)
 		(effects
 			(font
@@
 		)
 	)
-	(label "Xtal_in"
+	(label "Xtal_in_1"
 		(at 157.48 257.81 0)
 		(effects
@@
 		)
 	)
-	(label "Xtal_out"
+	(label "Xtal_out_2"
 		(at 125.73 259.08 0)
 		(effects
@@
 		)
 	)
-	(label "Xtal_out"
+	(label "Xtal_out_1"
 		(at 157.48 262.89 0)
 		(effects
@@
 			)
 		)
-		(property "Footprint" ""
+		(property "Footprint" "Capacitor_SMD:C_0402_1005Metric"
 			(at 107.95 264.16 0)
 			(effects
@@
 			)
 		)
-		(property "Footprint" ""
+		(property "Footprint" "Crystal:Crystal_SMD_3225-4Pin_3.2x2.5mm"
 			(at 170.18 185.42 0)
 			(effects
@@
 			)
 		)
-		(property "Footprint" ""
+		(property "Footprint" "Capacitor_SMD:C_0402_1005Metric"
 			(at 95.25 264.16 0)
 			(effects
@@
 			)
 		)
-		(property "Footprint" ""
+		(property "Footprint" "Resistor_SMD:R_0402_1005Metric"
 			(at 185.42 185.42 0)
 			(effects
@@
 			)
 		)
-		(property "Value" "33pF"
+		(property "Value" "15pF"
 			(at 166.37 191.7762 0)
 			(effects
@@
 			)
 		)
-		(property "Footprint" ""
+		(property "Footprint" "Capacitor_SMD:C_0402_1005Metric"
 			(at 163.83 190.5 0)
 			(effects
@@
 			)
 		)
-		(property "Value" "33pF"
+		(property "Value" "15pF"
 			(at 179.07 191.7762 0)
 			(effects
@@
 			)
 		)
-		(property "Footprint" ""
+		(property "Footprint" "Capacitor_SMD:C_0402_1005Metric"
 			(at 176.53 190.5 0)
 			(effects
@@
 			)
 		)
-		(property "Footprint" ""
+		(property "Footprint" "Crystal:Crystal_SMD_3225-4Pin_3.2x2.5mm"
 			(at 101.6 259.08 0)
 			(effects
@@
 			)
 		)
-		(property "Footprint" ""
+		(property "Footprint" "Resistor_SMD:R_0402_1005Metric"
 			(at 116.84 259.08 0)
 			(effects
